File: mic.kicad_pcb (KiCad board)
At the start: 2 copper layers, 50 x 50 mm, 46 parts, among them J1 AudioPlug3, J2 USB_C_Receptacle_USB2.0_16P, SW1 SW_Push, U1 TS5A3159ADBVR, U2 INA826AID, U3 PCM2902CDBR, U4 TLV70033_SOT23-5, U5 USBLC6-2SC6, Y1 12MHz

Commit message: needs via, otherwise should be done)
Connections:
- net /MIC_BIAS renamed Net-(C18-Pad1)
Changed lines of the file:
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@@
 			(layers "*.Cu" "*.Mask")
 			(remove_unused_layers no)
-			(net "/MIC_BIAS")
+			(net "Net-(C18-Pad1)")
 		)
 		(pad "2" thru_hole circle
@@
 			)
 		)
-		(property "LCSC" "C11337"
-			(at 0 0 0)
-			(unlocked yes)
-			(layer "F.Fab")
-			(hide yes)
-			(effects
-				(font
-					(size 1 1)
-					(thickness 0.15)
-				)
-			)
-		)
 		(property ki_fp_filters "SOT?23*")
 		(sheetname "/")
@@
 			(layers "*.Cu" "*.Mask")
 			(remove_unused_layers no)
-			(net "/MIC_BIAS")
+			(net "Net-(C18-Pad1)")
 			(pintype "passive")
 		)
@@
 			(layers "*.Cu" "*.Mask")
 			(remove_unused_layers no)
-			(net "/MIC_BIAS")
+			(net "Net-(C18-Pad1)")
 		)
 		(embedded_fonts no)
@@
 		(width 0.2)
 		(layer "F.Cu")
-		(net "/MIC_BIAS")
+		(net "Net-(C18-Pad1)")
 	)
 	(segment
@@
 		(width 0.2)
 		(layer "F.Cu")
-		(net "/MIC_BIAS")
+		(net "Net-(C18-Pad1)")
 	)
 	(segment
@@
 		(width 0.5)
 		(layer "F.Cu")
-		(net "/MIC_BIAS")
+		(net "Net-(C18-Pad1)")
 	)
 	(segment
@@
 		(width 0.5)
 		(layer "F.Cu")
-		(net "/MIC_BIAS")
+		(net "Net-(C18-Pad1)")
 	)
 	(segment
@@
 		(width 0.5)
 		(layer "F.Cu")
-		(net "/MIC_BIAS")
+		(net "Net-(C18-Pad1)")
 	)
 	(segment
@@
 		(width 0.2)
 		(layer "F.Cu")
-		(net "/MIC_BIAS")
+		(net "Net-(C18-Pad1)")
 	)
 	(via
@@
 		(drill 0.3)
 		(layers "F.Cu" "B.Cu")
-		(net "/MIC_BIAS")
+		(net "Net-(C18-Pad1)")
 	)
 	(segment
@@
 		(width 0.5)
 		(layer "B.Cu")
-		(net "/MIC_BIAS")
+		(net "Net-(C18-Pad1)")
 	)
 	(segment
@@
 		(width 0.5)
 		(layer "B.Cu")
-		(net "/MIC_BIAS")
+		(net "Net-(C18-Pad1)")
 	)
 	(segment
@@
 		(width 0.5)
 		(layer "B.Cu")
-		(net "/MIC_BIAS")
+		(net "Net-(C18-Pad1)")
 	)
 	(segment
