File: mic.kicad_pcb (KiCad board)
At the start: 2 copper layers, 50 x 50 mm, 46 parts, among them J1 AudioPlug3, J2 USB_C_Receptacle_USB2.0_16P, SW1 SW_Push, U1 TS5A3159ADBVR, U2 INA826AID, U3 PCM2902CDBR, U4 TLV70033_SOT23-5, U5 USBLC6-2SC6, Y1 12MHz

Commit message: final tht
Parts:
- added C21: 100n, Capacitor_THT:C_Disc_D3.4mm_W2.1mm_P2.50mm, F.Cu at (93.0, 113.0)
- added C22: 1u, Capacitor_THT:C_Disc_D3.4mm_W2.1mm_P2.50mm, F.Cu at (88.2, 113.0)
- added R18: 100k, Resistor_THT:R_Axial_DIN0204_L3.6mm_D1.6mm_P2.54mm_Vertical, F.Cu at (81.0, 110.8)
- added U6: 74LVC1G74DP, Package_SO:TSSOP-8_3x3mm_P0.65mm, F.Cu at (84.0, 113.0)
- R2: value 10k -> 100k
Connections:
- R2 pad 1: Net-(R2-Pad1) -> Net-(U6-C)
- R3 pad 2: Net-(R2-Pad1) -> Net-(U6-D)
- SW1 pad 2: Net-(R2-Pad1) -> Net-(U6-C)
- U1 pad 6: Net-(R2-Pad1) -> Net-(U6-D)
Routing:
- net Net-(U6-D): track 0.00 -> 71.7 mm, vias 0 -> 1
- net Net-(R2-Pad1): track 66.4 -> 0.00 mm
- net Net-(U6-C): track 0.00 -> 28.8 mm
- net Net-(U6-~{CLR}): track 0.00 -> 9.65 mm, vias 0 -> 1
- net +5V: track 86.0 -> 93.9 mm
- net Earth: track 0.00 -> 1.60 mm, vias 109 -> 98

Commit message: smd version, took only few hours
Parts:
- added C20: 100n, Capacitor_SMD:C_0603_1608Metric, F.Cu at (131.2, 113.2)
- added R9: 1k5R, Resistor_SMD:R_0603_1608Metric, B.Cu at (150.2, 102.0)
- C1, C10, C15, C16, C17, C18, C2, C21, C22, C3: footprint Capacitor_THT:C_Disc_D3.4mm_W2.1mm_P2.50mm -> Capacitor_SMD:C_0603_1608Metric
- C11, C12: footprint Capacitor_THT:CP_Radial_D8.0mm_P3.50mm -> Capacitor_SMD:CP_Elec_8x10
- C13, C14, C19, C4, C5, C6, C7, C8, C9: footprint Capacitor_THT:C_Disc_D3.4mm_W2.1mm_P2.50mm -> Capacitor_SMD:C_0603_1608Metric; moved to B.Cu
- J2: footprint Connector_USB:USB_C_Receptacle_G-Switch_GT-USB-7051x -> mic:USB_C_Receptacle_G-Switch_GT-USB-7051x_NoA8
- MK2: footprint AOM-5024L-HD-F-R:MIC_AOM-5024L-HD-F-R -> mic:MIC_AOM-5024L-HD-F-R
- R1, R11, R14, R18, R2, R3, R4, R5, R6: footprint Resistor_THT:R_Axial_DIN0204_L3.6mm_D1.6mm_P2.54mm_Vertical -> Resistor_SMD:R_0603_1608Metric
- R10, R12, R13, R15, R16, R7, R8: footprint Resistor_THT:R_Axial_DIN0204_L3.6mm_D1.6mm_P2.54mm_Vertical -> Resistor_SMD:R_0603_1608Metric; moved to B.Cu
- U2: footprint INA826AID:SOIC127P599X175-8N -> mic:SOIC127P599X175-8N
- U3: footprint PCM2902C:SOP65P780X200-28N -> mic:SOP65P780X200-28N
- Y1: footprint Crystal:Crystal_C26-LF_D2.1mm_L6.5mm_Vertical -> Crystal:Crystal_SMD_5032-2Pin_5.0x3.2mm; moved to B.Cu
- moved C15 65.5 mm to (146.2, 94.3)
- moved C17 63.8 mm to (151.0, 90.7)
- moved R14 63.4 mm to (158.0, 84.2), turned to 180 degrees
- moved R16 62.1 mm to (143.0, 103.3), turned to 90 degrees
- moved R13 60.5 mm to (138.1, 102.8), turned to 0 degrees
- moved C10 60.3 mm to (146.2, 95.8), turned to 0 degrees
- moved U2 60.2 mm to (151.5, 95.1)
- moved R11 60.1 mm to (154.7, 91.5), turned to 0 degrees
- moved C16 59.6 mm to (149.5, 90.8), turned to -90 degrees
- moved C2 58.1 mm to (141.1, 98.2)
- moved R6 56.8 mm to (146.2, 92.8), turned to 0 degrees
- moved R4 56.2 mm to (156.0, 96.5), turned to 90 degrees
- moved U1 56.2 mm to (154.8, 88.5), turned to 90 degrees
- moved C3 55.3 mm to (143.0, 92.5), turned to 180 degrees
- moved R12 55.0 mm to (138.1, 96.8)
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Routing:
- net Net-(C18-Pad1): track 29.2 -> 2.96 mm, vias 1 -> 0
- net Net-(U6-D): track 71.7 -> 47.9 mm, vias 1 -> 0
- net Net-(U6-C): track 28.8 -> 10.0 mm
- net Net-(U3-VOUTL): track 37.3 -> 19.1 mm, vias 0 -> 1
- net Net-(U2-RG_2): track 20.0 -> 2.08 mm
- net Net-(U3-VBUS): track 25.5 -> 7.52 mm, vias 2 -> 0
- net Net-(U3-D+): track 3.32 -> 17.4 mm
- net Net-(U3-VCCCI): track 14.5 -> 1.99 mm
- net Net-(U3-VINL): track 14.4 -> 2.62 mm, vias 1 -> 0
- net Net-(U2-+IN): track 14.5 -> 3.60 mm
- net +3.3V: track 25.1 -> 35.9 mm
- net +5V: track 93.9 -> 103.2 mm, vias 3 -> 4
- net /USB_DP: track 18.7 -> 9.73 mm, vias 3 -> 0
- net Net-(U2-REF): track 16.2 -> 7.32 mm
- net /USB_DM: track 18.0 -> 9.60 mm, vias 0 -> 3
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
Commit message: redoing the board
Parts:
- C11, C12: moved to B.Cu
- R15: moved to F.Cu
- moved C14 118.9 mm to (270.5, 68.2), turned to 0 degrees
- moved C13 118.8 mm to (270.8, 72.7), turned to 0 degrees
- moved Y1 118.2 mm to (267.0, 70.8)
- moved C7 117.7 mm to (259.5, 72.2), turned to 180 degrees
- moved C6 113.7 mm to (259.5, 69.2)
- moved C5 111.7 mm to (259.5, 67.9), turned to 180 degrees
- moved C8 111.3 mm to (259.5, 74.7)
- moved R10 110.9 mm to (264.0, 70.7)
- moved U3 110.9 mm to (252.5, 71.2)
- moved C9 110.1 mm to (245.5, 66.9)
- moved C4 110.1 mm to (245.5, 69.7)
- moved C19 109.9 mm to (245.2, 73.4)
- moved R16 106.9 mm to (245.2, 71.9), turned to 0 degrees
- moved R9 105.2 mm to (252.6, 77.4), turned to 0 degrees
- moved R8 104.4 mm to (239.2, 74.0)
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Routing:
- net +5V: track 103.2 -> 14.7 mm, vias 4 -> 0
- net Net-(U6-D): track 47.9 -> 2.46 mm
- net +3.3V: track 35.9 -> 2.58 mm, vias 1 -> 0
- net Net-(U3-VOUTL): track 19.1 -> 0.00 mm, vias 1 -> 0
- net Net-(U3-VOUTR): track 15.3 -> 0.00 mm, vias 1 -> 0
- net Net-(R4-Pad1): track 12.0 -> 0.00 mm
- net Net-(U2-RG_3): track 23.0 -> 13.2 mm
- net Net-(U3-D+): track 17.4 -> 8.81 mm
- net Net-(C10-Pad1): track 9.53 -> 1.52 mm, vias 1 -> 0
- net Net-(U3-VDDI): track 3.75 -> 9.07 mm
- net Net-(J2-CC2): track 11.0 -> 5.78 mm
- net Net-(U3-XTI): track 9.45 -> 14.7 mm
- net Net-(U3-VCCXI): track 6.80 -> 2.72 mm
- net Net-(U3-XTO): track 10.5 -> 14.5 mm
- net Net-(J2-CC1): track 7.96 -> 4.31 mm
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- added copper zone on F.Cu, net +5V
- removed copper zone on B.Cu, net Earth
- removed copper zone on F.Cu, net Earth

Commit message: it is stiched alright
Parts:
- C10, C15, C16, C17, R15, R4, R5, R6, U2: moved to B.Cu
- C11, C12: moved to F.Cu
- moved C13 137.5 mm to (137.4, 106.2), turned to 180 degrees
- moved C14 134.3 mm to (142.0, 107.0), turned to -90 degrees
- moved Y1 130.9 mm to (140.2, 103.3), turned to 180 degrees
- moved R10 127.2 mm to (140.3, 100.3), turned to 0 degrees
- moved C8 125.3 mm to (136.3, 97.4), turned to 90 degrees
- moved C7 123.3 mm to (138.8, 97.4), turned to 90 degrees
- moved C6 121.0 mm to (141.8, 97.4), turned to 90 degrees
- moved C5 119.8 mm to (143.4, 97.4), turned to 90 degrees
- moved R9 119.7 mm to (133.5, 90.5), turned to -90 degrees
- moved U3 114.4 mm to (139.8, 90.4), turned to -90 degrees
- moved C19 108.1 mm to (137.5, 83.1), turned to 90 degrees
- moved R16 106.7 mm to (139.0, 83.1), turned to -90 degrees
- moved C4 105.1 mm to (141.3, 83.4), turned to -90 degrees
- moved R7 104.5 mm to (134.8, 79.0), turned to 90 degrees
- moved C9 102.8 mm to (144.0, 83.4), turned to 90 degrees
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Routing:
- net +5V: track 14.7 -> 129.0 mm, vias 0 -> 6
- net Net-(U6-D): track 2.46 -> 30.2 mm
- net +3.3V: track 2.58 -> 27.9 mm, vias 0 -> 1
- net Net-(U2-+IN): track 1.81 -> 21.8 mm, vias 0 -> 1
- net Net-(U3-VOUTR): track 0.00 -> 20.0 mm, vias 0 -> 1
- net Net-(U3-VOUTL): track 0.00 -> 12.4 mm, vias 0 -> 1
- net Net-(U3-VINL): track 0.65 -> 8.02 mm
- net Net-(U2-RG_2): track 2.75 -> 9.28 mm
- net Net-(C1-Pad1): track 4.33 -> 10.6 mm, vias 0 -> 1
- net Net-(U3-D+): track 8.81 -> 13.2 mm
- net Net-(U3-D-): track 5.14 -> 7.31 mm
- net Net-(R4-Pad1): track 0.00 -> 2.00 mm
- net Net-(U3-XTI): track 14.7 -> 13.0 mm
- net Net-(U3-XTO): track 14.5 -> 12.9 mm
- net Net-(U2-RG_3): track 13.2 -> 11.9 mm
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- added copper zone on B.Cu, net Earth
- added copper zone on F.Cu, net Earth
- removed copper zone on F.Cu, net +5V

Commit message: fixed errors
Parts:
- added C23: 100n, Capacitor_SMD:C_0603_1608Metric, F.Cu at (132.1, 98.3)
- added U7: SN74LVC1G17DBVR, Package_TO_SOT_SMD:SOT-23-5, F.Cu at (133.0, 102.0)
- R1: value 1k2 -> 2k2
- R14: value 1k -> 470R
- moved C21 3.11 mm to (136.5, 102.0), turned to 0 degrees
- moved R2 1.03 mm to (136.5, 103.5), turned to 0 degrees
- moved R4 0.18 mm to (156.0, 93.6)
Connections:
- C21 pad 1: Net-(U6-C) -> /BTN_RC
- J2 pad A6: /USB_DP -> /_USB_DP
- J2 pad A7: /USB_DM -> /_USB_DM
- J2 pad B6: /USB_DP -> /_USB_DP
- J2 pad B7: /USB_DM -> /_USB_DM
- R2 pad 1: Net-(U6-C) -> /BTN_RC
- SW1 pad 2: Net-(U6-C) -> /BTN_RC
- U5 pad 1: /USB_DP -> /_USB_DP
- U5 pad 3: /USB_DM -> /_USB_DM
- U6 pad 1: Net-(U6-C) -> /BTN_CLK
Routing:
- net Net-(U6-C): track 13.2 -> 0.00 mm
- net /BTN_RC: track 0.00 -> 11.5 mm
- net /USB_DP: track 8.19 -> 1.79 mm
- net /USB_DM: track 8.17 -> 1.80 mm
- net +5V: track 129.0 -> 135.3 mm
- net /_USB_DP: track 0.00 -> 5.97 mm, vias 0 -> 2
- net /_USB_DM: track 0.00 -> 5.94 mm
- net /BTN_CLK: track 0.00 -> 2.96 mm
- net Net-(U2-RG_2): track 9.28 -> 8.53 mm
- net Earth: vias 483 -> 477
