File: mic.kicad_sch (KiCad schematic)
At the start: 38 parts, among them J1 AudioPlug3, J2 USB_C_Receptacle_USB2.0_16P, SW1 SW_Push, U1 TS5A3159ADBVR, U2 INA826AID, U3 PCM2902CDBR, U4 TLV70033_SOT23-5, Y1 12MHz

Commit message: Add mic-bias/VBUS filters, codec input R, USB ESD; stereo jack
- R14/C18 mic-bias RC filter, R15 codec input resistor
- R16/C19 VBUS filter for PCM2902C, U5 USBLC6-2SC6 on D+/D-
- J1 -> PJ-3920-3A stereo jack (custom footprint in mic.pretty)
- All passives THT; C3 moved next to LDO; reroutes under U3
- LCSC: J2 C2843970, U3 code removed; R3 1k
- review.md updated

Co-Authored-By: Claude Opus 5.5 <noreply@anthropic.com>
Parts:
- removed C11, C12: 470u, Capacitor_THT:CP_Radial_D8.0mm_P3.50mm, symbol Device:C
- added C11, C12: 470u, Capacitor_THT:CP_Radial_D8.0mm_P3.50mm, symbol Device:C_Polarized
- added C16, C17: 100n, Capacitor_THT:C_Disc_D3.4mm_W2.1mm_P2.50mm, symbol Device:C
- added C18: 10u, Capacitor_THT:C_Disc_D3.4mm_W2.1mm_P2.50mm, symbol Device:C
- added C19: 1u, Capacitor_THT:C_Disc_D3.4mm_W2.1mm_P2.50mm, symbol Device:C
- added R14, R15: 1k, Resistor_THT:R_Axial_DIN0204_L3.6mm_D1.6mm_P2.54mm_Vertical, symbol Device:R
- added R16: 2R2, Resistor_THT:R_Axial_DIN0204_L3.6mm_D1.6mm_P2.54mm_Vertical, symbol Device:R
- added U5: USBLC6-2SC6, Package_TO_SOT_SMD:SOT-23-6, symbol Power_Protection:USBLC6-2SC6
- J1: footprint Connector_Audio:Jack_3.5mm_QingPu_WQP-PJ398SM_Vertical_CircularHoles -> mic:Jack_3.5mm_KoreanHropartsElec_PJ-3920-3A_Vertical; LCSC C22355828 -> C707259
- R1: value 2k2 -> 1k2
- R3: value 150R -> 1kR
- U3: LCSC C2651869 -> (none)
- U4: LCSC alr -> C11337
Connections:
- net +3.3V: now also R14.1; no longer R1.1
- net +5V: now also C16.2, C17.2, R16.1, U5.5 (VBUS); no longer U3.3 (VBUS)
- net Earth: now also U1.3, C16.1, C17.1, C18.2, C19.2, U5.2 (GND)
- net USB_DP: now reaches J2.A6 (D+), J2.B6 (D+), R7.2
- net USB_DP: now also U5.1 (I/O1), U5.6 (I/O1)
- net USB_DM: now reaches J2.A7 (D-), J2.B7 (D-), R8.2
- net USB_DM: now also U5.3 (I/O2), U5.4 (I/O2)
- net at U3.12 (VINL), U3.13 (VINR): now also R15.2; no longer C10.1
- net at U3.16 (VOUTL): now also C11.1
- net at J1.T: now also C11.2
- net at U3.15 (VOUTR): now also C12.1
- net at J1.R: now also C12.2
- new net: C10.1, R15.1
- new net: C19.1, R16.2, U3.3 (VBUS)
- new net MIC_BIAS: C18.1, R1.1, R14.2
- no-connect marks 5 -> 4
